Commit message: Integrate ORB-SLAM3 stereo-inertial VIO into athena_description
- Add orb.launch.py to launch the ORB-SLAM3 stereo-inertial node
  alongside the existing Genesis bridge and Ackermann nodes
- Add config/ with ORB-SLAM3 camera+IMU calibration yaml and vocabulary
- Update genesis_launcher.py and URDF for ZED2i stereo/IMU topics
  consumed by ORB-SLAM3
- Update CMakeLists.txt to install new config/launch resources
- Add orb_slam3_ros2 and vision_opencv as workspace dependencies
- Remove unused ground_noise.png

File: src/athena_description/urdf/athena_rover-6.urdf.xacro (robot description, xacro)
@@ -178,5 +178,5 @@
     <origin xyz="0.0 0.0 -0.111" rpy="0 0 0"/>
     <axis xyz="0 0 1"/>
-    <limit lower="-0.79" upper="0.79" effort="10" velocity="1.0"/>
+    <limit lower="-1.57" upper="1.57" effort="10" velocity="1.0"/>
     <dynamics damping="0.2" friction="0.05"/>
   </joint>
@@ -209,5 +209,5 @@
     <axis xyz="0 1 0"/>
     <dynamics damping="0.01" friction="0.05"/>
-      <limit upper="3.14"/>
+      <limit upper="3.14" velocity="10.0" effort="100.0"/>
   </joint>
   <!-- ================================================================ -->
@@ -270,5 +270,5 @@
     <origin xyz="0.0 0.0 -0.111" rpy="0 0 0"/>
     <axis xyz="0 0 1"/>
-    <limit lower="-0.7854" upper="0.7854" effort="10" velocity="1.0"/>
+    <limit lower="-1.57" upper="1.57" effort="10" velocity="1.0"/>
     <dynamics damping="0.2" friction="0.05"/>
   </joint>
@@ -361,5 +361,5 @@
     <origin xyz="0.0 0.0 -0.111" rpy="0 0 0"/>
     <axis xyz="0 0 1"/>
-    <limit lower="-0.7854" upper="0.7854" effort="10" velocity="1.0"/>
+    <limit lower="-1.57" upper="1.57" effort="10" velocity="1.0"/>
     <dynamics damping="0.2" friction="0.05"/>
   </joint>
@@ -452,5 +452,5 @@
     <origin xyz="0.0 0.0 -0.111" rpy="0 0 0"/>
     <axis xyz="0 0 1"/>
-    <limit lower="-0.7854" upper="0.7854" effort="10" velocity="1.0"/>
+    <limit lower="-1.57" upper="1.57" effort="10" velocity="1.0"/>
     <dynamics damping="0.2" friction="0.05"/>
   </joint>
