Commit message: Add Livox Mid360 URDF data to incorporate with the existing rover

File: src/athena_description/urdf/athena_rover-6 copy.urdf (robot description, URDF)
Before this commit: robot athena_rover, 23 links, 22 joints
Links:
- link livox_mid360_link: geometry visual mesh filename=package://athena_description/meshes/visual/livox-mid-360-as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 scale=0.001 0.001 0.001

File: src/athena_description/urdf/athena_rover-6.urdf.xacro (robot description, xacro)
@@ -4,8 +4,5 @@
 <!-- Package path: package://athena_description/meshes/                          -->
 <robot xmlns:xacro="http://www.ros.org/wiki/xacro" name="athena_rover">
-  <xacro:include filename="$(find zed_wrapper)/urdf/zed_macro.urdf.xacro"/>
-  <xacro:zed_camera name="zed2i" model="zed2i" enable_gnss="false">
-    <origin xyz="0 0 0" rpy="0 0 0"/>
-  </xacro:zed_camera>
+  ⁠<xacro:include filename="$(find athena_description)/urdf/livox_mid360.xacro"/>
   <material name="aluminium">
     <color rgba="0.75 0.75 0.80 1.0"/>
@@ -55,4 +52,33 @@
     <origin xyz="0.2 0 0.3" rpy="0 0 0"/>
   </joint>
+  <link name="livox_mid360_link">
+    <visual>
+      <origin xyz="0.0 0.0 0.0" rpy="1.5708 0 0"/>
+      <geometry>
+        <mesh filename="package://athena_description/meshes/visual/livox-mid-360-asm.stl"
+              scale="0.001 0.001 0.001"/>
+      </geometry>
+      <material name="aluminium"/>
+    </visual>
+    <collision>
+      <origin xyz="0.0 0.0 0.0" rpy="1.5708 0 0"/>
+      <geometry>
+        <mesh filename="package://athena_description/meshes/collision/livox-mid-360-asm.stl"
+              scale="0.001 0.001 0.001"/>
+      </geometry>
+    </collision>
+    <inertial>
+      <mass value="1.2"/>
+      <origin xyz="0.00 0.00 0.00" rpy="0 0 0"/>
+      <inertia ixx="1e-4" ixy="1e-4" ixz="1e-4"
+               iyy="1e-4" iyz="1e-4"
+               izz="1e-4"/>
+    </inertial>
+  </link>
+  <joint name="livox_mid360_joint" type="fixed">
+    <parent link="base_link"/>
+    <child link="livox_mid360_link"/>
+    <origin xyz="0 0 0.175" rpy="0 0 0"/>
+  </joint>
   <link name="bogey_left">
     <visual>

Commit message: Fix hardcoded ZED mesh paths to work irrespective of ROS distro

File: src/athena_description/urdf/athena_rover-6 copy.urdf (robot description, URDF)
Before this commit: robot athena_rover, 23 links, 22 joints
Links:
- link zed2i_camera_center: geometry collision mesh filename=package://zed_description/meshes/zed2i.stl; visual mesh filename=package://zed_description/meshes/zed2i.stl

File: src/athena_description/urdf/athena_rover-6.urdf (robot description, URDF)
Before this commit: robot athena_rover, 23 links, 22 joints
Links:
- link zed2i_camera_center: geometry collision mesh filename=package://zed_description/meshes/zed2i.stl; visual mesh filename=package://zed_description/meshes/zed2i.stl
