Commit message: feat: getting VIO

File: src/athena_description/urdf/athena_rover-6.urdf (robot description, URDF)
Before this commit: robot athena_rover, 22 links, 21 joints
Links:
- link zed2i_camera_center: mass None -> 0
Joints:
- joint zed2i_right_camera_joint_optical: origin xyz=0 0 0 rpy=0 0.0 0 -> xyz=0 0 0 rpy=-1.5707963267948966 0.0 -1.5707963267948966

Commit message: feat: Added Independent steering(Ackermann)

File: src/athena_description/urdf/athena_rover-6.urdf (robot description, URDF)
Before this commit: robot athena_rover, 22 links, 21 joints
Joints:
- joint steer_front_left: limit lower=-0.79 upper=0.79 effort=10 velocity=1.0 -> lower=-1.57 upper=1.57 effort=10 velocity=1.0
- joint steer_front_right: limit lower=-0.7854 upper=0.7854 effort=10 velocity=1.0 -> lower=-1.57 upper=1.57 effort=10 velocity=1.0
- joint steer_rear_left: limit lower=-0.7854 upper=0.7854 effort=10 velocity=1.0 -> lower=-1.57 upper=1.57 effort=10 velocity=1.0
- joint steer_rear_right: limit lower=-0.7854 upper=0.7854 effort=10 velocity=1.0 -> lower=-1.57 upper=1.57 effort=10 velocity=1.0

Commit message: Add Livox Mid-360 as URDF link

File: src/athena_description/urdf/athena_rover-6.urdf (robot description, URDF)
Before this commit: robot athena_rover, 22 links, 21 joints
Links:
- added link livox_mid360_link, mass 0.265; visual cylinder length=0.05 radius=0.03
Joints:
- added joint livox_mid360_joint: type fixed, parent base_link, child livox_mid360_link, origin xyz=0 0 0.08 rpy=0 0 0

Commit message: Modify inertia values to satisfy eigenvalue conditions

File: src/athena_description/urdf/athena_rover-6.urdf (robot description, URDF)
Before this commit: robot athena_rover, 23 links, 22 joints
Links:
- link livox_mid360_link: geometry visual mesh filename=package://athena_description/meshes/visual/livox-mid-360-as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 scale=0.001 0.001 0.001

File: src/athena_description/urdf/athena_rover-6.urdf.xacro (robot description, xacro)
@@ -71,6 +71,6 @@
       <mass value="1.2"/>
       <origin xyz="0.00 0.00 0.00" rpy="0 0 0"/>
-      <inertia ixx="1e-4" ixy="1e-4" ixz="1e-4"
-               iyy="1e-4" iyz="1e-4"
+      <inertia ixx="1e-4" ixy="0.0" ixz="0.0"
+           iyy="1e-4" iyz="0.0"
                izz="1e-4"/>
     </inertial>

Commit message: Fix ZED 2i position in space

File: src/athena_description/urdf/athena_rover-6.urdf (robot description, URDF)
Before this commit: robot athena_rover, 23 links, 22 joints
Joints:
- joint zed2i_mount_joint: origin xyz=0.2 0 0.3 rpy=0 0 0 -> xyz=0.2 0 0.1 rpy=0 0 0

File: src/athena_description/urdf/athena_rover-6.urdf.xacro (robot description, xacro)
@@ -79,5 +79,5 @@
     <parent link="base_link"/>
     <child link="livox_mid360_link"/>
-    <origin xyz="0 0 0.175" rpy="0 0 0"/>
+    <origin xyz="0 0 0.175" rpy="3.1416 0 0"/>
   </joint>
   <link name="bogey_left">

Commit message: feat: Add all 3 types of steering, added both rtabmap and orbslam code(just in case)

File: src/athena_description/urdf/athena_rover-6.urdf (robot description, URDF)
Before this commit: robot athena_rover, 22 links, 21 joints
Joints:
- joint zed2i_left_camera_joint: origin xyz=-0.01 0.06 0 rpy=0 0 0 -> xyz=-0.01 0.06 0 rpy=0 3.1415 0

Commit message: Added Terrain: Known issue: 	1. Rover is flipping radomly 	2. Orbslam did not work

File: src/athena_description/urdf/athena_rover-6.urdf (robot description, URDF)
Before this commit: robot athena_rover, 22 links, 21 joints
Joints:
- joint steer_rear_right: limit lower=-1.57 upper=1.57 effort=10 velocity=1.0 -> lower=-1.57 upper=1.57 effort=1000 velocity=1.0

Commit message: refactor: Made the code more modular and changed the directory structure.
- Created the genesis_bridge folder to replace the genesis_launcher.py which contained all the code that we wrote.

fix: fixed a few naming errors in the urdf and a few minor bugs in all three seering modes

feat(vio): removed orbslam3 and replaced it with rtabmap.

-- known bugs: (getting the vio data with major errors)

File: src/athena_description/urdf/athena_rover-6.urdf (robot description, URDF)
Before this commit: robot athena_rover, 22 links, 21 joints
Joints:
- joint steer_front_right: limit lower=-1.57 upper=1.57 effort=10 velocity=1.0 -> lower=-1.57 upper=1.57 effort=1000 velocity=1.0
- joint steer_housing_mount_front_left: origin xyz=-0.39291 0.11681 0.0425000 rpy=0 0 0 -> xyz=0.34458 0.10398 0.0425000 rpy=0 0 0
- joint steer_housing_mount_front_right: origin xyz=-0.39291 -0.11681 0.0425000 rpy=0 0 0 -> xyz=0.34458 -0.10398 0.0425000 rpy=0 0 0
- joint steer_housing_mount_rear_left: origin xyz=0.34458 0.10398 0.0425000 rpy=0 0 0 -> xyz=-0.39291 0.11681 0.0425000 rpy=0 0 0
- joint steer_housing_mount_rear_right: origin xyz=0.34458 -0.10398 0.0425000 rpy=0 0 0 -> xyz=-0.39291 -0.11681 0.0425000 rpy=0 0 0
- joint steer_rear_right: limit lower=-1.57 upper=1.57 effort=1000 velocity=1.0 -> lower=-1.57 upper=1.57 effort=10 velocity=1.0
- joint wheel_front_left_spin: limit upper=3.14 effort=100.0 velocity=10.0 -> (none)
- joint wheel_rear_left_spin: limit (none) -> upper=3.14 effort=100.0 velocity=10.0

File: src/athena_description/urdf/athena_rover-6.urdf.xacro (robot description, xacro)
@@ -120,94 +120,83 @@
   </joint>
   <!-- ================================================================ -->
-  <!-- FRONT-LEFT: steering split into housing (fixed) + coupler (steers) -->
+  <!-- FRONT-LEFT -->
   <!-- ================================================================ -->
   <link name="steer_housing_front_left">
     <visual>
-      <origin xyz="0.6145 -1.1306 -0.1077" rpy="0 0 3.1416"/>
-      <geometry>
-        <mesh filename="package://athena_description/meshes/visual/SteeringMotorHousing.stl"
-              scale="0.001 0.001 0.001"/>
-      </geometry>
-      <material name="motor_grey"/>
-    </visual>
-    <collision>
-      <origin xyz="0.6145 -1.1306 -0.1077" rpy="0 0 3.1416"/>
-      <geometry>
-        <mesh filename="package://athena_description/meshes/collision/SteeringMotorHousing.stl"
-              scale="0.001 0.001 0.001"/>
+      <origin rpy="0 0 3.1416" xyz="0.6145 -1.1306 -0.1077"/>
+      <geometry>
+        <mesh filename="package://athena_description/meshes/visual/SteeringMotorHousing.stl" scale="0.001 0.001 0.001"/>
+      </geometry>
+      <material name="motor_grey"/>
+    </visual>
+    <collision>
+      <origin rpy="0 0 3.1416" xyz="0.6145 -1.1306 -0.1077"/>
+      <geometry>
+        <mesh filename="package://athena_description/meshes/collision/SteeringMotorHousing.stl" scale="0.001 0.001 0.001"/>
       </geometry>
     </collision>
     <inertial>
       <mass value="0.2"/>
-      <inertia ixx="0.0001" ixy="0" ixz="0"
-               iyy="0.0001" iyz="0"
-               izz="0.00005"/>
+      <inertia ixx="0.0001" ixy="0" ixz="0" iyy="0.0001" iyz="0" izz="0.00005"/>
     </inertial>
   </link>
   <joint name="steer_housing_mount_front_left" type="fixed">
     <parent link="bogey_left"/>
-    <child  link="steer_housing_front_left"/>
-    <origin xyz="-0.39291 0.11681 0.0425000" rpy="0 0 0"/>
+    <child link="steer_housing_front_left"/>
+    <origin rpy="0 0 0" xyz="-0.39291 0.11681 0.0425000"/>
   </joint>
   <link name="steer_coupler_front_left">
     <visual>
-      <origin xyz="-0.6145 1.1307 0.0063" rpy="0 0 0"/>
-      <geometry>
-        <mesh filename="package://athena_description/meshes/visual/stearing.stl"
-              scale="0.001 0.001 0.001"/>
-      </geometry>
-      <material name="motor_grey"/>
-    </visual>
-    <collision>
-      <origin xyz="-0.6145 1.1307 0.0063" rpy="0 0 0"/>
-      <geometry>
-        <mesh filename="package://athena_description/meshes/collision/stearing.stl"
-              scale="0.001 0.001 0.001"/>
+      <origin rpy="0 0 0" xyz="-0.6145 1.1307 0.0063"/>
+      <geometry>
+        <mesh filename="package://athena_description/meshes/visual/stearing.stl" scale="0.001 0.001 0.001"/>
+      </geometry>
+      <material name="motor_grey"/>
+    </visual>
+    <collision>
+      <origin rpy="0 0 0" xyz="-0.6145 1.1307 0.0063"/>
+      <geometry>
+        <mesh filename="package://athena_description/meshes/collision/stearing.stl" scale="0.001 0.001 0.001"/>
       </geometry>
     </collision>
     <inertial>
       <mass value="0.15"/>
-      <inertia ixx="0.0001" ixy="0" ixz="0"
-               iyy="0.0001" iyz="0"
-               izz="0.00005"/>
+      <inertia ixx="0.0001" ixy="0" ixz="0" iyy="0.0001" iyz="0" izz="0.00005"/>
     </inertial>
   </link>
   <joint name="steer_front_left" type="revolute">
     <parent link="steer_housing_front_left"/>
-    <child  link="steer_coupler_front_left"/>
-    <origin xyz="0.0 0.0 -0.111" rpy="0 0 0"/>
+    <child link="steer_coupler_front_left"/>
+    <origin rpy="0 0 0" xyz="0.0 0.0 -0.111"/>
     <axis xyz="0 0 1"/>
-    <limit lower="-1.57" upper="1.57" effort="10" velocity="1.0"/>
+    <limit effort="10" lower="-1.57" upper="1.57" velocity="1.0"/>
     <dynamics damping="0.2" friction="0.05"/>
   </joint>
   <link name="wheel_front_left">
     <visual>
-      <origin xyz="0.4497 0.3642 0.1895" rpy="0 0 0"/>
-      <geometry>
-        <mesh filename="package://athena_description/meshes/visual/wheel.stl"
-              scale="0.001 0.001 0.001"/>
+      <origin rpy="0 0 0" xyz="0.4497 0.3642 0.1895"/>
+      <geometry>
+        <mesh filename="package://athena_description/meshes/visual/wheel.stl" scale="0.001 0.001 0.001"/>
       </geometry>
       <material name="rubber"/>
     </visual>
     <collision>
-      <origin xyz="0 0 0" rpy="1.5708 0 0"/>
-      <geometry>
-        <cylinder radius="0.115" length="0.080"/>
+      <origin rpy="1.5708 0 0" xyz="0 0 0"/>
+      <geometry>
+        <cylinder length="0.080" radius="0.115"/>
       </geometry>
     </collision>
     <inertial>
       <mass value="0.8"/>
-      <inertia ixx="0.006" ixy="0" ixz="0"
-               iyy="0.010" iyz="0"
-               izz="0.006"/>
+      <inertia ixx="0.006" ixy="0" ixz="0" iyy="0.010" iyz="0" izz="0.006"/>
     </inertial>
   </link>
   <joint name="wheel_front_left_spin" type="continuous">
     <parent link="steer_coupler_front_left"/>
-    <child  link="wheel_front_left"/>
-    <origin xyz="0.0 0.0 -0.186" rpy="0 0 0"/>
+    <child link="wheel_front_left"/>
+    <origin rpy="0 0 0" xyz="0.0 0.0 -0.186"/>
     <axis xyz="0 1 0"/>
     <dynamics damping="0.01" friction="0.05"/>
-      <limit upper="3.14" velocity="10.0" effort="100.0"/>
+    <limit upper="3.14" velocity="10.0" effort="100.0"/>
   </joint>
   <!-- ================================================================ -->
@@ -216,87 +205,76 @@
   <link name="steer_housing_rear_left">
     <visual>
-      <origin xyz="-1.1029 0.6629 -0.1077" rpy="0 0 0.5317"/>
-      <geometry>
-        <mesh filename="package://athena_description/meshes/visual/SteeringMotorHousing.stl"
-              scale="0.001 0.001 0.001"/>
-      </geometry>
-      <material name="motor_grey"/>
-    </visual>
-    <collision>
-      <origin xyz="-1.1029 0.6629 -0.1077" rpy="0 0 0.5317"/>
-      <geometry>
-        <mesh filename="package://athena_description/meshes/collision/SteeringMotorHousing.stl"
-              scale="0.001 0.001 0.001"/>
+      <origin rpy="0 0 0.5317" xyz="-1.1029 0.6629 -0.1077"/>
+      <geometry>
+        <mesh filename="package://athena_description/meshes/visual/SteeringMotorHousing.stl" scale="0.001 0.001 0.001"/>
+      </geometry>
+      <material name="motor_grey"/>
+    </visual>
+    <collision>
+      <origin rpy="0 0 0.5317" xyz="-1.1029 0.6629 -0.1077"/>
+      <geometry>
+        <mesh filename="package://athena_description/meshes/collision/SteeringMotorHousing.stl" scale="0.001 0.001 0.001"/>
       </geometry>
     </collision>
     <inertial>
       <mass value="0.2"/>
-      <inertia ixx="0.0001" ixy="0" ixz="0"
-               iyy="0.0001" iyz="0"
-               izz="0.00005"/>
+      <inertia ixx="0.0001" ixy="0" ixz="0" iyy="0.0001" iyz="0" izz="0.00005"/>
     </inertial>
   </link>
   <joint name="steer_housing_mount_rear_left" type="fixed">
     <parent link="bogey_left"/>
-    <child  link="steer_housing_rear_left"/>
-    <origin xyz="0.34458 0.10398 0.0425000" rpy="0 0 0"/>
+    <child link="steer_housing_rear_left"/>
+    <origin rpy="0 0 0" xyz="0.34458 0.10398 0.0425000"/>
   </joint>
   <link name="steer_coupler_rear_left">
     <visual>
-      <origin xyz="-0.6145 1.1307 0.0063" rpy="0 0 0"/>
-      <geometry>
-        <mesh filename="package://athena_description/meshes/visual/stearing.stl"
-              scale="0.001 0.001 0.001"/>
-      </geometry>
-      <material name="motor_grey"/>
-    </visual>
-    <collision>
-      <origin xyz="-0.6145 1.1307 0.0063" rpy="0 0 0"/>
-      <geometry>
-        <mesh filename="package://athena_description/meshes/collision/stearing.stl"
-              scale="0.001 0.001 0.001"/>
+      <origin rpy="0 0 0" xyz="-0.6145 1.1307 0.0063"/>
+      <geometry>
+        <mesh filename="package://athena_description/meshes/visual/stearing.stl" scale="0.001 0.001 0.001"/>
+      </geometry>
+      <material name="motor_grey"/>
+    </visual>
+    <collision>
+      <origin rpy="0 0 0" xyz="-0.6145 1.1307 0.0063"/>
+      <geometry>
+        <mesh filename="package://athena_description/meshes/collision/stearing.stl" scale="0.001 0.001 0.001"/>
       </geometry>
     </collision>
     <inertial>
       <mass value="0.15"/>
-      <inertia ixx="0.0001" ixy="0" ixz="0"
-               iyy="0.0001" iyz="0"
-               izz="0.00005"/>
+      <inertia ixx="0.0001" ixy="0" ixz="0" iyy="0.0001" iyz="0" izz="0.00005"/>
     </inertial>
   </link>
   <joint name="steer_rear_left" type="revolute">
     <parent link="steer_housing_rear_left"/>
-    <child  link="steer_coupler_rear_left"/>
-    <origin xyz="0.0 0.0 -0.111" rpy="0 0 0"/>
+    <child link="steer_coupler_rear_left"/>
+    <origin rpy="0 0 0" xyz="0.0 0.0 -0.111"/>
     <axis xyz="0 0 1"/>
-    <limit lower="-1.57" upper="1.57" effort="10" velocity="1.0"/>
+    <limit effort="10" lower="-1.57" upper="1.57" velocity="1.0"/>
     <dynamics damping="0.2" friction="0.05"/>
   </joint>
   <link name="wheel_rear_left">
     <visual>
-      <origin xyz="0.4497 0.3642 0.1895" rpy="0 0 0"/>
-      <geometry>
-        <mesh filename="package://athena_description/meshes/visual/wheel.stl"
-              scale="0.001 0.001 0.001"/>
+      <origin rpy="0 0 0" xyz="0.4497 0.3642 0.1895"/>
+      <geometry>
+        <mesh filename="package://athena_description/meshes/visual/wheel.stl" scale="0.001 0.001 0.001"/>
       </geometry>
       <material name="rubber"/>
     </visual>
     <collision>
-      <origin xyz="0 0 0" rpy="1.5708 0 0"/>
-      <geometry>
-        <cylinder radius="0.115" length="0.080"/>
+      <origin rpy="1.5708 0 0" xyz="0 0 0"/>
+      <geometry>
+        <cylinder length="0.080" radius="0.115"/>
       </geometry>
     </collision>
     <inertial>
       <mass value="0.8"/>
-      <inertia ixx="0.006" ixy="0" ixz="0"
-               iyy="0.010" iyz="0"
-               izz="0.006"/>
+      <inertia ixx="0.006" ixy="0" ixz="0" iyy="0.010" iyz="0" izz="0.006"/>
     </inertial>
   </link>
   <joint name="wheel_rear_left_spin" type="continuous">
     <parent link="steer_coupler_rear_left"/>
-    <child  link="wheel_rear_left"/>
-    <origin xyz="0.0 0.0 -0.186" rpy="0 0 0"/>
+    <child link="wheel_rear_left"/>
+    <origin rpy="0 0 0" xyz="0.0 0.0 -0.186"/>
     <axis xyz="0 1 0"/>
     <dynamics damping="0.01" friction="0.05"/>
@@ -307,87 +285,76 @@
   <link name="steer_housing_front_right">
     <visual>
-      <origin xyz="1.1002 -0.6674 -0.1077" rpy="0 0 3.6692"/>
-      <geometry>
-        <mesh filename="package://athena_description/meshes/visual/SteeringMotorHousing.stl"
-              scale="0.001 0.001 0.001"/>
-      </geometry>
-      <material name="motor_grey"/>
-    </visual>
-    <collision>
-      <origin xyz="1.1002 -0.6674 -0.1077" rpy="0 0 3.6692"/>
-      <geometry>
-        <mesh filename="package://athena_description/meshes/collision/SteeringMotorHousing.stl"
-              scale="0.001 0.001 0.001"/>
+      <origin rpy="0 0 3.6692" xyz="1.1002 -0.6674 -0.1077"/>
+      <geometry>
+        <mesh filename="package://athena_description/meshes/visual/SteeringMotorHousing.stl" scale="0.001 0.001 0.001"/>
+      </geometry>
+      <material name="motor_grey"/>
+    </visual>
+    <collision>
+      <origin rpy="0 0 3.6692" xyz="1.1002 -0.6674 -0.1077"/>
+      <geometry>
+        <mesh filename="package://athena_description/meshes/collision/SteeringMotorHousing.stl" scale="0.001 0.001 0.001"/>
       </geometry>
     </collision>
     <inertial>
       <mass value="0.2"/>
-      <inertia ixx="0.0001" ixy="0" ixz="0"
-               iyy="0.0001" iyz="0"
-               izz="0.00005"/>
+      <inertia ixx="0.0001" ixy="0" ixz="0" iyy="0.0001" iyz="0" izz="0.00005"/>
     </inertial>
   </link>
   <joint name="steer_housing_mount_front_right" type="fixed">
     <parent link="bogey_right"/>
-    <child  link="steer_housing_front_right"/>
-    <origin xyz="-0.39291 -0.11681 0.0425000" rpy="0 0 0"/>
+    <child link="steer_housing_front_right"/>
+    <origin rpy="0 0 0" xyz="-0.39291 -0.11681 0.0425000"/>
   </joint>
   <link name="steer_coupler_front_right">
     <visual>
-      <origin xyz="0.6145 -1.1307 0.0063" rpy="0 0 3.1416"/>
-      <geometry>
-        <mesh filename="package://athena_description/meshes/visual/stearing.stl"
-              scale="0.001 0.001 0.001"/>
-      </geometry>
-      <material name="motor_grey"/>
-    </visual>
-    <collision>
-      <origin xyz="0.6145 -1.1307 0.0063" rpy="0 0 3.1416"/>
-      <geometry>
-        <mesh filename="package://athena_description/meshes/collision/stearing.stl"
-              scale="0.001 0.001 0.001"/>
+      <origin rpy="0 0 3.1416" xyz="0.6145 -1.1307 0.0063"/>
+      <geometry>
+        <mesh filename="package://athena_description/meshes/visual/stearing.stl" scale="0.001 0.001 0.001"/>
+      </geometry>
+      <material name="motor_grey"/>
+    </visual>
+    <collision>
+      <origin rpy="0 0 3.1416" xyz="0.6145 -1.1307 0.0063"/>
+      <geometry>
+        <mesh filename="package://athena_description/meshes/collision/stearing.stl" scale="0.001 0.001 0.001"/>
       </geometry>
     </collision>
     <inertial>
       <mass value="0.15"/>
-      <inertia ixx="0.0001" ixy="0" ixz="0"
-               iyy="0.0001" iyz="0"
-               izz="0.00005"/>
+      <inertia ixx="0.0001" ixy="0" ixz="0" iyy="0.0001" iyz="0" izz="0.00005"/>
     </inertial>
   </link>
   <joint name="steer_front_right" type="revolute">
     <parent link="steer_housing_front_right"/>
-    <child  link="steer_coupler_front_right"/>
-    <origin xyz="0.0 0.0 -0.111" rpy="0 0 0"/>
+    <child link="steer_coupler_front_right"/>
+    <origin rpy="0 0 0" xyz="0.0 0.0 -0.111"/>
     <axis xyz="0 0 1"/>
-    <limit lower="-1.57" upper="1.57" effort="10" velocity="1.0"/>
+    <limit effort="10" lower="-1.57" upper="1.57" velocity="1.0"/>
     <dynamics damping="0.2" friction="0.05"/>
   </joint>
   <link name="wheel_front_right">
     <visual>
-      <origin xyz="-0.4497 -0.3642 0.1895" rpy="0 0 3.1416"/>
-      <geometry>
-        <mesh filename="package://athena_description/meshes/visual/wheel.stl"
-              scale="0.001 0.001 0.001"/>
+      <origin rpy="0 0 3.1416" xyz="-0.4497 -0.3642 0.1895"/>
+      <geometry>
+        <mesh filename="package://athena_description/meshes/visual/wheel.stl" scale="0.001 0.001 0.001"/>
       </geometry>
       <material name="rubber"/>
     </visual>
     <collision>
-      <origin xyz="0 0 0" rpy="1.5708 0 0"/>
-      <geometry>
-        <cylinder radius="0.115" length="0.080"/>
+      <origin rpy="1.5708 0 0" xyz="0 0 0"/>
+      <geometry>
+        <cylinder length="0.080" radius="0.115"/>
       </geometry>
     </collision>
     <inertial>
       <mass value="0.8"/>
-      <inertia ixx="0.006" ixy="0" ixz="0"
-               iyy="0.010" iyz="0"
-               izz="0.006"/>
+      <inertia ixx="0.006" ixy="0" ixz="0" iyy="0.010" iyz="0" izz="0.006"/>
     </inertial>
   </link>
   <joint name="wheel_front_right_spin" type="continuous">
     <parent link="steer_coupler_front_right"/>
-    <child  link="wheel_front_right"/>
-    <origin xyz="0.0 0.0 -0.186" rpy="0 0 0"/>
+    <child link="wheel_front_right"/>
+    <origin rpy="0 0 0" xyz="0.0 0.0 -0.186"/>
     <axis xyz="0 1 0"/>
     <dynamics damping="0.01" friction="0.05"/>
@@ -398,87 +365,76 @@
   <link name="steer_housing_rear_right">
     <visual>
-      <origin xyz="-0.6145 1.1306 -0.1077" rpy="0 0 0"/>
-      <geometry>
-        <mesh filename="package://athena_description/meshes/visual/SteeringMotorHousing.stl"
-              scale="0.001 0.001 0.001"/>
-      </geometry>
-      <material name="motor_grey"/>
-    </visual>
-    <collision>
-      <origin xyz="-0.6145 1.1306 -0.1077" rpy="0 0 0"/>
-      <geometry>
-        <mesh filename="package://athena_description/meshes/collision/SteeringMotorHousing.stl"
-              scale="0.001 0.001 0.001"/>
+      <origin rpy="0 0 0" xyz="-0.6145 1.1306 -0.1077"/>
+      <geometry>
+        <mesh filename="package://athena_description/meshes/visual/SteeringMotorHousing.stl" scale="0.001 0.001 0.001"/>
+      </geometry>
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